File: CM5_HighSpeed.kicad_sch (KiCad schematic)
At the start: 1 part, among them J501 Hirose DF40C-100DS-0.4V

Commit message: Added USB connector for flashing eMMC and related switches
Parts:
- added J601: Conn_01x02_Pin, Connector_PinHeader_2.54mm:PinHeader_1x02_P2.54mm_Vertical, symbol Connector:Conn_01x02_Pin
Connections:
- net GND: now also J601.2 (Pin_2)
- net KEY/RECOVERY: now reaches J501.226 (SARADC_VIN0_KEY/RECOVERY)
- net KEY/RECOVERY: now also J601.1 (Pin_1)
- net USB2_HOST2_DP: now reaches J501.263 (USB2_HOST2_DP)
- net USB2_HOST2_DM: now reaches J501.265 (USB2_HOST2_DM)
- net USB_OTG0_VBUSDET: now reaches J501.297 (USB_OTG0_VBUSDET)
- no-connect marks 53 -> 49
