File: Power_12_to_5_8.kicad_sch (KiCad schematic)
At the start: 14 parts, among them J401 PJ-102AH

Commit message: Update to fix power connection mistakes in both IWCD and HK configurations. For IWCD added bridge rectifier diodes needed for PoE, for HK updated to look at correct ref voltage for the 12V generation DC/DC, rotated the TVS to correct orientation and updated input diodes to be >=100V
Parts:
- renumbered C403 to C401, C405 to C402, C401 to C403, C402 to C405, R402 to R401, R401 to R402
Changed lines of the file:
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@@
 		(dnp no)
 		(fields_autoplaced yes)
-		(property "Reference" "C405"
+		(property "Reference" "C402"
 			(at 68.58 130.8099 0)
 			(effects
@@
 			(project "cm5_unified_carrier"
 				(path "/ee887ca3-c545-439a-9405-8d7a48a3d148/6259954f-99d8-4c66-ab9f-731a7dc153d0"
-					(reference "C405")
+					(reference "C402")
 					(unit 1)
 				)
@@
 		(dnp no)
 		(fields_autoplaced yes)
-		(property "Reference" "#PWR0406"
+		(property "Reference" "#PWR0407"
 			(at 224.79 144.78 0)
 			(effects
@@
 			(project "cm5_unified_carrier"
 				(path "/ee887ca3-c545-439a-9405-8d7a48a3d148/6259954f-99d8-4c66-ab9f-731a7dc153d0"
-					(reference "#PWR0406")
+					(reference "#PWR0407")
 					(unit 1)
 				)
@@
 		(dnp no)
 		(fields_autoplaced yes)
-		(property "Reference" "#PWR0407"
+		(property "Reference" "#PWR0406"
 			(at 200.66 53.34 0)
 			(effects
@@
 			(project ""
 				(path "/ee887ca3-c545-439a-9405-8d7a48a3d148/6259954f-99d8-4c66-ab9f-731a7dc153d0"
-					(reference "#PWR0407")
+					(reference "#PWR0406")
 					(unit 1)
 				)
@@
 		(dnp no)
 		(fields_autoplaced yes)
-		(property "Reference" "#PWR0403"
+		(property "Reference" "#PWR0404"
 			(at 177.8 142.24 0)
 			(effects
@@
 			(project "cm5_unified_carrier"
 				(path "/ee887ca3-c545-439a-9405-8d7a48a3d148/6259954f-99d8-4c66-ab9f-731a7dc153d0"
-					(reference "#PWR0403")
+					(reference "#PWR0404")
 					(unit 1)
 				)
@@
 		(dnp no)
 		(fields_autoplaced yes)
-		(property "Reference" "#PWR0402"
+		(property "Reference" "#PWR0405"
 			(at 187.96 66.04 0)
 			(effects
@@
 			(project "cm5_unified_carrier"
 				(path "/ee887ca3-c545-439a-9405-8d7a48a3d148/6259954f-99d8-4c66-ab9f-731a7dc153d0"
-					(reference "#PWR0402")
+					(reference "#PWR0405")
 					(unit 1)
 				)
@@
 		(dnp no)
 		(fields_autoplaced yes)
-		(property "Reference" "#PWR0405"
+		(property "Reference" "#PWR0401"
 			(at 33.02 142.24 0)
 			(effects
@@
 			(project "cm5_unified_carrier"
 				(path "/ee887ca3-c545-439a-9405-8d7a48a3d148/6259954f-99d8-4c66-ab9f-731a7dc153d0"
-					(reference "#PWR0405")
+					(reference "#PWR0401")
 					(unit 1)
 				)
@@
 		(dnp no)
 		(fields_autoplaced yes)
-		(property "Reference" "R402"
+		(property "Reference" "R401"
 			(at 161.29 140.9699 0)
 			(effects
@@
 			(project "cm5_unified_carrier"
 				(path "/ee887ca3-c545-439a-9405-8d7a48a3d148/6259954f-99d8-4c66-ab9f-731a7dc153d0"
-					(reference "R402")
+					(reference "R401")
 					(unit 1)
 				)
@@
 		(dnp no)
 		(fields_autoplaced yes)
-		(property "Reference" "C403"
+		(property "Reference" "C401"
 			(at 36.83 129.9209 0)
 			(effects
@@
 			(project ""
 				(path "/ee887ca3-c545-439a-9405-8d7a48a3d148/6259954f-99d8-4c66-ab9f-731a7dc153d0"
-					(reference "C403")
+					(reference "C401")
 					(unit 1)
 				)
@@
 		(dnp no)
 		(fields_autoplaced yes)
-		(property "Reference" "C401"
+		(property "Reference" "C403"
 			(at 83.82 51.1809 0)
 			(effects
@@
 			(project ""
 				(path "/ee887ca3-c545-439a-9405-8d7a48a3d148/6259954f-99d8-4c66-ab9f-731a7dc153d0"
-					(reference "C401")
+					(reference "C403")
 					(unit 1)
 				)
@@
 		(dnp no)
 		(fields_autoplaced yes)
-		(property "Reference" "#PWR0404"
+		(property "Reference" "#PWR0402"
 			(at 64.77 142.24 0)
 			(effects
@@
 			(project "cm5_unified_carrier"
 				(path "/ee887ca3-c545-439a-9405-8d7a48a3d148/6259954f-99d8-4c66-ab9f-731a7dc153d0"
-					(reference "#PWR0404")
+					(reference "#PWR0402")
 					(unit 1)
 				)
@@
 		(dnp no)
 		(fields_autoplaced yes)
-		(property "Reference" "#PWR0401"
+		(property "Reference" "#PWR0403"
 			(at 80.01 63.5 0)
 			(effects
@@
 			(project ""
 				(path "/ee887ca3-c545-439a-9405-8d7a48a3d148/6259954f-99d8-4c66-ab9f-731a7dc153d0"
-					(reference "#PWR0401")
+					(reference "#PWR0403")
 					(unit 1)
 				)
@@
 		(dnp no)
 		(fields_autoplaced yes)
-		(property "Reference" "R401"
+		(property "Reference" "R402"
 			(at 170.18 69.8499 0)
 			(effects
@@
 			(project ""
 				(path "/ee887ca3-c545-439a-9405-8d7a48a3d148/6259954f-99d8-4c66-ab9f-731a7dc153d0"
-					(reference "R401")
+					(reference "R402")
 					(unit 1)
 				)
@@
 		(dnp no)
 		(fields_autoplaced yes)
-		(property "Reference" "C402"
+		(property "Reference" "C405"
 			(at 191.77 52.0699 0)
 			(effects
@@
 			(project "cm5_unified_carrier"
 				(path "/ee887ca3-c545-439a-9405-8d7a48a3d148/6259954f-99d8-4c66-ab9f-731a7dc153d0"
-					(reference "C402")
+					(reference "C405")
 					(unit 1)
 				)
